File: SmartDrv.kicad_pcb (KiCad board)
At the start: 4 copper layers, 60 x 60 mm, 99 parts, among them J1 Conn_01x04, J2 Conn_01x02, J3 Conn_01x02, J4 Conn_01x02, J5 Conn_01x02, J6 Conn_01x02, J7 Conn_01x03, Q1 BSC040N10NS5, Q2 BSC040N10NS5, Q3 BSC040N10NS5, Q4 BSC040N10NS5, Q6 NPN, Q7 Si2319CDS, U1 IR2104, U2 IR2104, U3 AT32F423CBT7, U4 MCP6002-xSN, U5 TJA1051T, U6 AMS1117-5.0, U7 AP2112K-3.3, U8 L7812, U9 KF7.62-2P, Y1 Crystal_GND24

Commit message: Add files via upload
Routing:
- net +5V: track 112.8 -> 114.7 mm
- net +12V: track 125.3 -> 126.4 mm
- net GND: track 2.87 -> 3.88 mm, vias 98 -> 96

Commit message: Add files via upload
Parts:
- removed Q6: NPN, Package_TO_SOT_SMD:SOT-23
- added C32: 100n, Capacitor_SMD:C_0603_1608Metric, F.Cu at (227.9, 52.2)
- added C33: 100n, Capacitor_SMD:C_0603_1608Metric, F.Cu at (232.4, 52.2)
- added D19: 1N5819WS, Diode_SMD:D_SOD-323, F.Cu at (220.1, 58.1)
- added F1: Fuse, Fuse:Fuse_1812_4532Metric, B.Cu at (247.3, 62.0)
- added F2: Fuse, Fuse:Fuse_1812_4532Metric, B.Cu at (241.2, 62.0)
- added F3: Fuse, Fuse:Fuse_1812_4532Metric, B.Cu at (218.0, 61.7)
- added F4: Fuse, Fuse:Fuse_1812_4532Metric, B.Cu at (212.4, 61.8)
- added Q5: 2N7002K, Package_TO_SOT_SMD:SOT-23, F.Cu at (214.8, 58.1)
Connections:
- U3 pad 46: unconnected-(U3-PB9-Pad46) -> Buzz
Routing:
- net Buzz: track 0.00 -> 15.9 mm, vias 0 -> 2
- net +5V: track 114.7 -> 121.1 mm, vias 3 -> 6
- net Net-(BZ1--): track 2.94 -> 7.07 mm
- net R_shunt_1: track 23.6 -> 19.7 mm
- net GND: track 3.88 -> 6.80 mm, vias 96 -> 97
- net Net-(Q5-G): track 2.13 -> 4.35 mm
- net Current 2: track 17.7 -> 17.1 mm
- net Current 1: track 22.0 -> 22.6 mm
- added copper zone on B.Cu, net V_IN
- removed copper zone on B.Cu, net GND
