File: SmartDrv.kicad_sch (KiCad schematic)
At the start: 106 parts, among them J1 Conn_01x04, J2 Conn_01x02, J3 Conn_01x02, J4 Conn_01x02, J5 Conn_01x02, J6 Conn_01x02, J7 Conn_01x03, Q1 BSC040N10NS5, Q2 BSC040N10NS5, Q3 BSC040N10NS5, Q4 BSC040N10NS5, Q5 PMOS, Q6 NPN, U1 IR2104, U2 IR2104, U3 AT32F423CBT7, U4 MCP6002-xSN, U5 TJA1051T, U6 AMS1117-5.0, U7 AP2112K-3.3, U8 L7812, U9 KF7.62-2P, Y1 Crystal_GND24

Commit message: Add files via upload
Parts:
- D15: value SMAJ6.0A -> SMAJ15.0A
- R12: value 20k -> 15k
- R22, R23, R24, R25: value 10 -> 1M
Other:
- moved on the sheet: R1
Changed lines of the file:
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@@
 	(wire
 		(pts
-			(xy 88.9 43.18) (xy 100.33 43.18)
+			(xy 88.9 43.18) (xy 95.25 43.18)
 		)
 		(stroke
@@
 	(wire
 		(pts
+			(xy 102.87 43.18) (xy 107.95 43.18)
+		)
+		(stroke
+			(width 0)
+			(type default)
+		)
+	)
+	(wire
+		(pts
 			(xy 222.25 257.81) (xy 234.95 257.81)
 		)
@@
 	(symbol
 		(lib_id "Device:R")
-		(at 104.14 43.18 270)
+		(at 99.06 43.18 270)
 		(unit 1)
 		(exclude_from_sim no)
@@
 		(fields_autoplaced yes)
 		(property "Reference" "R1"
-			(at 104.14 36.83 90)
+			(at 99.06 36.83 90)
 			(effects
 				(font
@@
 		)
 		(property "Value" "R"
-			(at 104.14 39.37 90)
+			(at 99.06 39.37 90)
 			(effects
 				(font
@@
 		)
 		(property "Footprint" "Resistor_SMD:R_0805_2012Metric"
-			(at 104.14 41.402 90)
+			(at 99.06 41.402 90)
 			(effects
 				(font
@@
 		)
 		(property "Datasheet" "~"
-			(at 104.14 43.18 0)
+			(at 99.06 43.18 0)
 			(effects
 				(font
@@
 		)
 		(property "Description" "Resistor"
-			(at 104.14 43.18 0)
+			(at 99.06 43.18 0)
 			(effects
 				(font
@@
 			)
 		)
-		(property "Value" "10"
+		(property "Value" "1M"
 			(at 196.088 93.98 90)
 			(effects
@@
 			)
 		)
-		(property "Value" "20k"
+		(property "Value" "15k"
 			(at 170.18 146.05 90)
 			(effects
@@
 		(on_board yes)
 		(dnp no)
-		(fields_autoplaced yes)
 		(property "Reference" "D15"
 			(at 311.15 139.6999 90)
@@
 			)
 		)
-		(property "Value" "SMAJ6.0A"
-			(at 311.15 142.2399 90)
+		(property "Value" "SMAJ15.0A"
+			(at 309.118 144.272 90)
 			(effects
 				(font
@@
 			)
 		)
-		(property "Description" "400W unidirectional Transient Voltage Suppressor, 6.0Vr, SMA(DO-214AC)"
+		(property "Description" "400W unidirectional Transient Voltage Suppressor, 15.0Vr, SMA(DO-214AC)"
 			(at 308.61 140.97 0)
 			(effects
@@
 			)
 		)
-		(property "Value" "10"
+		(property "Value" "1M"
 			(at 207.772 30.48 90)
 			(effects
@@
 			)
 		)
-		(property "Value" "10"
+		(property "Value" "1M"
 			(at 268.478 93.98 90)
 			(effects
@@
 			)
 		)
-		(property "Value" "10"
+		(property "Value" "1M"
 			(at 271.018 29.972 0)
 			(effects

Commit message: Add files via upload
Parts:
- removed D3, D4, D6, D7: 1N5819, Diode_SMD:D_SMA, symbol Diode:1N5819
- added D13, D18: SS110, Diode_SMD:D_SMA, symbol Diode:SS110
- added D3, D4, D6, D7: SS310, Diode_SMD:D_SMA, symbol Diode:SS310
- D15: value SMAJ15.0A -> SMAJ30.0A
Connections:
- net +12V: now also D13.2 (A), D18.2 (A)
- net +5V: now also U4.8 (V+); no longer U4.4 (V-)
- net GND: now also U4.4 (V-); no longer U4.8 (V+)
- net R_shunt_1: now also D4.2 (A)
- net R_shunt_2: now also Q3.1 (S), Q3.2 (S), Q3.3 (S), D6.2 (A); no longer Q3.5 (D)
- net V_IN: now also Q2.5 (D), D3.1 (K), D7.1 (K); no longer Q2.1 (S), Q2.2 (S), Q2.3 (S)
- net at C8.2, Q1.1 (S), Q1.2 (S)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: now also D3.2 (A), D4.1 (K)
- net at C8.1, U1.8 (VB): now also D13.1 (K)
- net at C9.1, U2.8 (VB): now also D18.1 (K)
- new net: C9.2, D6.1 (K), D7.2 (A), Q2.1 (S), Q2.2 (S), Q2.3 (S), Q3.5 (D), U2.6 (VS), U9.2
Other:
- moved on the sheet: Q2, Q3, U4C

Commit message: Add files via upload
Parts:
- removed Q5: PMOS, Package_TO_SOT_SMD:SOT-23, symbol Simulation_SPICE:PMOS
- added Q7: Si2319CDS, Package_TO_SOT_SMD:SOT-23, symbol Transistor_FET:Si2319CDS
Connections:
- net VCC: now also Q7.2 (S)
- net V_IN: now also Q7.3 (D)
- net at D17.2 (A), R13.1: now also Q7.1 (G)
Other:
- moved on the sheet: D17
Changed lines of the file:
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@@
 	)
 	(junction
-		(at 283.21 146.05)
-		(diameter 0)
-		(color 0 0 0 0)
-	)
-	(junction
 		(at 285.75 50.8)
 		(diameter 0)
@@
 	)
 	(junction
+		(at 280.67 137.16)
+		(diameter 0)
+		(color 0 0 0 0)
+	)
+	(junction
 		(at 215.9 58.42)
 		(diameter 0)
@@
 	)
 	(junction
-		(at 283.21 137.16)
-		(diameter 0)
-		(color 0 0 0 0)
-	)
-	(junction
 		(at 101.6 146.05)
 		(diameter 0)
@@
 	)
 	(junction
+		(at 280.67 146.05)
+		(diameter 0)
+		(color 0 0 0 0)
+	)
+	(junction
 		(at 78.74 146.05)
 		(diameter 0)
@@
 	(wire
 		(pts
+			(xy 280.67 146.05) (xy 271.78 146.05)
+		)
+		(stroke
+			(width 0)
+			(type default)
+		)
+	)
+	(wire
+		(pts
 			(xy 247.65 237.49) (xy 260.35 237.49)
 		)
@@
 	(wire
 		(pts
-			(xy 283.21 146.05) (xy 271.78 146.05)
+			(xy 283.21 146.05) (xy 280.67 146.05)
 		)
 		(stroke
@@
 	(wire
 		(pts
-			(xy 276.86 137.16) (xy 283.21 137.16)
+			(xy 276.86 137.16) (xy 280.67 137.16)
 		)
 		(stroke
@@
 	(wire
 		(pts
-			(xy 283.21 144.78) (xy 283.21 146.05)
+			(xy 280.67 144.78) (xy 280.67 146.05)
 		)
 		(stroke
@@
 	(wire
 		(pts
-			(xy 283.21 137.16) (xy 295.91 137.16)
-		)
-		(stroke
-			(width 0)
-			(type default)
-		)
-	)
-	(wire
-		(pts
 			(xy 153.67 148.59) (xy 158.75 148.59)
 		)
@@
 	(wire
 		(pts
+			(xy 280.67 137.16) (xy 295.91 137.16)
+		)
+		(stroke
+			(width 0)
+			(type default)
+		)
+	)
+	(wire
+		(pts
 			(xy 269.24 60.96) (xy 294.64 60.96)
 		)
@@
 	(symbol
 		(lib_id "Diode:BZT52Bxx")
-		(at 283.21 140.97 270)
+		(at 280.67 140.97 270)
 		(unit 1)
 		(exclude_from_sim no)
@@
 		(fields_autoplaced yes)
 		(property "Reference" "D17"
-			(at 285.75 139.6999 90)
+			(at 283.21 139.6999 90)
 			(effects
 				(font
@@
 		)
 		(property "Value" "BZT52Bxx"
-			(at 285.75 142.2399 90)
+			(at 283.21 142.2399 90)
 			(effects
 				(font
@@
 		)
 		(property "Footprint" "Diode_SMD:D_SOD-123F"
-			(at 278.765 140.97 0)
+			(at 276.225 140.97 0)
 			(effects
 				(font
@@
 		)
 		(property "Datasheet" "https://diotec.com/tl_files/diotec/files/pdf/datasheets/bzt52b2v4.pdf"
-			(at 283.21 140.97 0)
+			(at 280.67 140.97 0)
 			(effects
 				(font
@@
 		)
 		(property "Description" "500mW Zener Diode, SOD-123F"
-			(at 283.21 140.97 0)
+			(at 280.67 140.97 0)
 			(effects
 				(font
@@
 	)
 	(symbol
-		(lib_name "PMOS_1")
-		(lib_id "Simulation_SPICE:PMOS")
-		(at 271.78 139.7 90)
-		(unit 1)
-		(exclude_from_sim no)
-		(in_bom yes)
-		(on_board yes)
-		(dnp no)
-		(property "Reference" "Q5"
-			(at 279.146 144.526 90)
-			(effects
-				(font
-					(size 1.27 1.27)
-				)
-				(justify left)
-			)
-		)
-		(property "Value" "PMOS"
-			(at 279.146 141.986 90)
-			(effects
-				(font
-					(size 1.27 1.27)
-				)
-				(justify left)
-			)
-		)
-		(property "Footprint" "Package_TO_SOT_SMD:SOT-23"
-			(at 269.24 134.62 0)
-			(effects
-				(font
-					(size 1.27 1.27)
-				)
-				(hide yes)
-			)
-		)
-		(property "Datasheet" "https://ngspice.sourceforge.io/docs/ngspice-html-manual/manual.xhtml#cha_MOSFETs"
-			(at 284.48 139.7 0)
-			(effects
-				(font
-					(size 1.27 1.27)
-				)
-				(hide yes)
-			)
-		)
-		(property "Description" "P-MOSFET transistor, drain/source/gate"
-			(at 271.78 139.7 0)
-			(effects
-				(font
-					(size 1.27 1.27)
-				)
-				(hide yes)
-			)
-		)
-		(property "Sim.Device" "PMOS"
-			(at 288.925 139.7 0)
-			(effects
-				(font
-					(size 1.27 1.27)
-				)
-				(hide yes)
-			)
-		)
-		(property "Sim.Type" "VDMOS"
-			(at 290.83 139.7 0)
-			(effects
-				(font
-					(size 1.27 1.27)
-				)
-				(hide yes)
-			)
-		)
-		(property "Sim.Pins" "1=G 2=D 3=S"
-			(at 287.02 139.7 0)
-			(effects
-				(font
-					(size 1.27 1.27)
-				)
-				(hide yes)
-			)
-		)
-		(pin "2"
-		)
-		(pin "1"
-		)
-		(pin "3"
-		)
-		(instances
-			(project "SmartDrv"
-				(path "/e4f5a07e-eede-42da-a027-6e670981fa18"
-					(reference "Q5")
-					(unit 1)
-				)
-			)
-		)
-	)
-	(symbol
 		(lib_id "power:GND")
 		(at 63.5 208.28 0)
@@
 					(unit 1)
 				)
+			)
+		)
+	)
+	(symbol
+		(lib_id "Transistor_FET:Si2319CDS")
+		(at 271.78 139.7 90)
+		(unit 1)
+		(exclude_from_sim no)
+		(in_bom yes)
+		(on_board yes)
+		(dnp no)
+		(fields_autoplaced yes)
+		(property "Reference" "Q7"
+			(at 271.78 130.81 90)
+			(effects
+				(font
+					(size 1.27 1.27)
+				)
+			)
+		)
+		(property "Value" "Si2319CDS"
+			(at 271.78 133.35 90)
+			(effects
+				(font
+					(size 1.27 1.27)
+				)
+			)
+		)
+		(property "Footprint" "Package_TO_SOT_SMD:SOT-23"
+			(at 273.685 134.62 0)
+			(effects
+				(font
+					(size 1.27 1.27)
+					(italic yes)
+				)
+				(justify left)
+				(hide yes)
+			)
+		)
+		(property "Datasheet" "http://www.vishay.com/docs/66709/si2319cd.pdf"
+			(at 275.59 134.62 0)
+			(effects
+				(font
+					(size 1.27 1.27)
+				)
+				(justify left)
+				(hide yes)
+			)
+		)
+		(property "Description" "-4.4A Id, -40V Vds, P-Channel MOSFET, SOT-23"
+			(at 271.78 139.7 0)
+			(effects
+				(font
+					(size 1.27 1.27)
+				)
+				(hide yes)
+			)
+		)
+		(pin "1"
+		)
+		(pin "3"
+		)
+		(pin "2"
+		)
+		(instances
+			(project "SmartDrv"
+				(path "/e4f5a07e-eede-42da-a027-6e670981fa18"
+					(reference "Q7")
+					(unit 1)
+				)

Commit message: Add files via upload
Parts:
- removed Q6: NPN, Package_TO_SOT_SMD:SOT-23, symbol Simulation_SPICE:NPN
- added D19: 1N5819WS, Diode_SMD:D_SOD-323, symbol Diode:1N5819WS
- added F1, F2, F3, F4: Fuse, Fuse:Fuse_1812_4532Metric, symbol Device:Fuse
- added Q5: 2N7002K, Package_TO_SOT_SMD:SOT-23, symbol Transistor_FET:2N7002K
Connections:
- net +3V3: no longer C32.1, C33.1, C34.1, C35.1
- net +5V: now also C32.1, C33.1, C34.1, C35.1, D19.1 (K)
- net Buzz: now also U3.46 (PB9)
- net GND: now also Q5.2 (S)
- net V_IN: now also F1.1, F1.2, F2.1, F2.2, F3.1, F3.2, F4.1, F4.2
- net at R15.2: now also Q5.1 (G)
- net at BZ1.2 (-): now also D19.2 (A), Q5.3 (D)
Other:
- moved on the sheet: C32, C33, C34, C35, R15
